File: Hardware/PCB/voltproc/voltproc.kicad_pcb (KiCad board)
At the start: 2 copper layers, 0 parts

Commit message: reorg schematic, RC and linear lag
Parts:
- added C1: 10uF, ao_tht:CP_Radial_D6.3mm_P2.50mm, B.Cu at (103.8, 18.7)
- added C10: 100nF, ao_tht:C_Disc_D3.0mm_W1.6mm_P2.50mm, B.Cu at (122.9, 121.6)
- added C11: 20pF, ao_tht:C_Disc_D3.0mm_W1.6mm_P2.50mm, B.Cu at (97.5, 21.3)
- added C12: 20pF, ao_tht:C_Disc_D3.0mm_W1.6mm_P2.50mm, B.Cu at (77.1, 47.9)
- added C13: 200pF, ao_tht:C_Disc_D3.0mm_W1.6mm_P2.50mm, B.Cu at (97.5, 44.1)
- added C14: 200pF, ao_tht:C_Disc_D3.0mm_W1.6mm_P2.50mm, B.Cu at (77.1, 21.3)
- added C15: 100nF, ao_tht:C_Disc_D3.0mm_W1.6mm_P2.50mm, B.Cu at (94.9, 32.7)
- added C16: 100nF, ao_tht:C_Disc_D3.0mm_W1.6mm_P2.50mm, B.Cu at (77.2, 32.7)
- added C2: 10uF, ao_tht:CP_Radial_D6.3mm_P2.50mm, B.Cu at (86.0, 18.7)
- added C3: 47pF, ao_tht:C_Disc_D3.0mm_W1.6mm_P2.50mm, B.Cu at (105.1, 125.4)
- added C4: 220nF, ao_tht:C_Disc_D3.0mm_W1.6mm_P2.50mm, B.Cu at (126.7, 121.6)
- added C5: 2.2uF, ao_tht:C_Radial_D8.0mm_H11.5mm_P3.50mm, B.Cu at (122.9, 114.0)
- added C6: 1uF, ao_tht:C_Disc_D3.0mm_W1.6mm_P2.50mm, B.Cu at (77.2, 110.2)
- added C7: 100nF, ao_tht:C_Disc_D3.0mm_W1.6mm_P2.50mm, B.Cu at (95.0, 117.8)
- added C8: 100nF, ao_tht:C_Disc_D3.0mm_W1.6mm_P2.50mm, B.Cu at (77.1, 117.8)
- added C9: 100nF, ao_tht:C_Disc_D3.0mm_W1.6mm_P2.50mm, B.Cu at (105.1, 117.8)
- added D1: 1N5817, ao_tht:D_DO-41_SOD81_P10.16mm_Horizontal, B.Cu at (108.9, 18.7)
- added D2: 1N5817, ao_tht:D_DO-41_SOD81_P10.16mm_Horizontal, B.Cu at (119.0, 23.0)
- added GRAF1: Holes, voltproc:voltproc_panel_holes, F.Cu at (200.0, 100.0)
- added J1: Synth_power_2x5, ao_tht:Power_Header, B.Cu at (127.9, 32.7)
- added J10: Jack, ao_tht:Jack_6.35mm_PJ_629HAN_slots, F.Cu at (75.0, 60.0)
- added J11: Jack, ao_tht:Jack_6.35mm_PJ_629HAN_slots, F.Cu at (100.0, 60.0)
- added J12: Jack, ao_tht:Jack_6.35mm_PJ_629HAN_slots, F.Cu at (75.0, 175.0)
- added J13: Jack, ao_tht:Jack_6.35mm_PJ_629HAN_slots, F.Cu at (75.0, 85.0)
- added J14: Jack, ao_tht:Jack_6.35mm_PJ_629HAN_slots, F.Cu at (100.0, 85.0)
- added J15: Jack, ao_tht:Jack_6.35mm_PJ_629HAN_slots, F.Cu at (75.0, 150.0)
- added J16: Jack, ao_tht:Jack_6.35mm_PJ_629HAN_slots, F.Cu at (125.0, 60.0)
- added J17: Jack, ao_tht:Jack_6.35mm_PJ_629HAN_slots, F.Cu at (125.0, 85.0)
- added J18: Jack, ao_tht:Jack_6.35mm_PJ_629HAN_slots, F.Cu at (100.0, 150.0)
- added J19: Jack, ao_tht:Jack_6.35mm_PJ_629HAN_slots, F.Cu at (100.0, 175.0)
- added J2: 2_pin_Molex_header, ao_tht:Molex_KK-254_AE-6410-02A_1x02_P2.54mm_Vertical, B.Cu at (116.5, 46.7)
- added J3: 2_pin_Molex_header, ao_tht:Molex_KK-254_AE-6410-02A_1x02_P2.54mm_Vertical, B.Cu at (108.9, 46.7)
- added J4: Conn_01x13, Connector_PinHeader_2.54mm:PinHeader_1x13_P2.54mm_Vertical, F.Cu at (91.0, 98.5)
- added J7: Conn_01x13, Connector_PinSocket_2.54mm:PinSocket_1x13_P2.54mm_Vertical, B.Cu at (191.0, 98.5)
- added J8: Jack, ao_tht:Jack_6.35mm_PJ_629HAN_slots, F.Cu at (125.0, 150.0)
- added J9: Jack, ao_tht:Jack_6.35mm_PJ_629HAN_slots, F.Cu at (125.0, 175.0)
- added R1: 100k, ao_tht:R_Axial_DIN0207_L6.3mm_D2.5mm_P10.16mm_Horizontal, B.Cu at (105.1, 110.2)
- added R10: 100k, ao_tht:R_Axial_DIN0207_L6.3mm_D2.5mm_P10.16mm_Horizontal, B.Cu at (120.3, 126.4)
- added R11: 1k, ao_tht:R_Axial_DIN0207_L6.3mm_D2.5mm_P10.16mm_Horizontal, B.Cu at (120.3, 130.5)
- added R12: 2.7k, ao_tht:R_Axial_DIN0207_L6.3mm_D2.5mm_P10.16mm_Horizontal, B.Cu at (84.8, 102.5)
- added R13: 15k, ao_tht:R_Axial_DIN0207_L6.3mm_D2.5mm_P10.16mm_Horizontal, B.Cu at (69.5, 102.5)
- added R14: 2.7k, ao_tht:R_Axial_DIN0207_L6.3mm_D2.5mm_P10.16mm_Horizontal, B.Cu at (91.1, 72.1)
- added R15: 15k, ao_tht:R_Axial_DIN0207_L6.3mm_D2.5mm_P10.16mm_Horizontal, B.Cu at (67.0, 72.1)
- added R16: 100k, ao_tht:R_Axial_DIN0207_L6.3mm_D2.5mm_P10.16mm_Horizontal, B.Cu at (105.1, 28.9)
- added R17: 100k, ao_tht:R_Axial_DIN0207_L6.3mm_D2.5mm_P10.16mm_Horizontal, B.Cu at (119.0, 35.2)
- added R18: 100k, ao_tht:R_Axial_DIN0207_L6.3mm_D2.5mm_P10.16mm_Horizontal, B.Cu at (119.0, 27.6)
- added R19: 100k, ao_tht:R_Axial_DIN0207_L6.3mm_D2.5mm_P10.16mm_Horizontal, B.Cu at (119.0, 31.4)
- added R2: 10k, ao_tht:R_Axial_DIN0207_L6.3mm_D2.5mm_P10.16mm_Horizontal, B.Cu at (105.1, 114.0)
- added R20: 100k, ao_tht:R_Axial_DIN0207_L6.3mm_D2.5mm_P10.16mm_Horizontal, B.Cu at (69.5, 44.1)
- added R21: 100k, ao_tht:R_Axial_DIN0207_L6.3mm_D2.5mm_P10.16mm_Horizontal, B.Cu at (69.5, 36.5)
- added R22: 100k, ao_tht:R_Axial_DIN0207_L6.3mm_D2.5mm_P10.16mm_Horizontal, B.Cu at (94.9, 25.1)
- added R23: 100k, ao_tht:R_Axial_DIN0207_L6.3mm_D2.5mm_P10.16mm_Horizontal, B.Cu at (79.7, 40.3)
- added R24: 10k, ao_tht:R_Axial_DIN0207_L6.3mm_D2.5mm_P10.16mm_Horizontal, B.Cu at (105.1, 36.5)
- added R25: 10k, ao_tht:R_Axial_DIN0207_L6.3mm_D2.5mm_P10.16mm_Horizontal, B.Cu at (69.5, 28.9)
- added R26: 10k, ao_tht:R_Axial_DIN0207_L6.3mm_D2.5mm_P10.16mm_Horizontal, B.Cu at (94.9, 40.3)
- added R27: 10k, ao_tht:R_Axial_DIN0207_L6.3mm_D2.5mm_P10.16mm_Horizontal, B.Cu at (79.7, 25.1)
- added R28: 1k, ao_tht:R_Axial_DIN0207_L6.3mm_D2.5mm_P10.16mm_Horizontal, B.Cu at (121.6, 47.9)
- added R29: 1k, ao_tht:R_Axial_DIN0207_L6.3mm_D2.5mm_P10.16mm_Horizontal, B.Cu at (121.6, 44.1)
- added R3: 10k, ao_tht:R_Axial_DIN0207_L6.3mm_D2.5mm_P10.16mm_Horizontal, B.Cu at (94.9, 106.3)
- added R30: 1k, ao_tht:R_Axial_DIN0207_L6.3mm_D2.5mm_P10.16mm_Horizontal, B.Cu at (94.9, 133.0)
- added R31: 1k, ao_tht:R_Axial_DIN0207_L6.3mm_D2.5mm_P10.16mm_Horizontal, B.Cu at (94.9, 136.8)
- added R4: 10M, ao_tht:R_Axial_DIN0207_L6.3mm_D2.5mm_P10.16mm_Horizontal, B.Cu at (105.1, 121.6)
- added R5: 68k, ao_tht:R_Axial_DIN0207_L6.3mm_D2.5mm_P10.16mm_Horizontal, B.Cu at (105.1, 129.2)
- added R6: 20k, ao_tht:R_Axial_DIN0207_L6.3mm_D2.5mm_P10.16mm_Horizontal, B.Cu at (69.5, 121.6)
- added R7: 4.7k, ao_tht:R_Axial_DIN0207_L6.3mm_D2.5mm_P10.16mm_Horizontal, B.Cu at (79.7, 129.2)
- added R8: 200R, ao_tht:R_Axial_DIN0207_L6.3mm_D2.5mm_P10.16mm_Horizontal, B.Cu at (79.7, 133.0)
- added R9: 10k, ao_tht:R_Axial_DIN0207_L6.3mm_D2.5mm_P10.16mm_Horizontal, B.Cu at (79.7, 125.4)
- added RV1: B100k, ao_tht:Potentiometer_Alpha_16mm_Single_Vertical, F.Cu at (225.0, 119.0)
- added RV4: B1M, ao_tht:Potentiometer_Alpha_16mm_Dual_Vertical, F.Cu at (175.0, 119.0)
- added SW1: SW_DPDT_x2, ao_tht:DPDT-toggle-switch-1M-seriesx, F.Cu at (200.0, 110.0)
- added SW2: SW_DPDT_x2, ao_tht:DPDT-toggle-switch-1M-seriesx, F.Cu at (200.0, 128.0)
- added TP1: -12V, ao_tht:TestPoint_THTPad_D1.5mm_Drill0.7mm, B.Cu at (69.5, 16.2)
- added TP2: +12V, ao_tht:TestPoint_THTPad_D1.5mm_Drill0.7mm, B.Cu at (79.7, 16.2)
- added TP3: GND, ao_tht:TestPoint_THTPad_1.5x1.5mm_Drill0.7mm, B.Cu at (74.6, 16.2)
- added U1: TL074, ao_tht:DIP-14_W7.62mm_Socket_LongPads, B.Cu at (91.1, 25.1)
- added U2: TL074, ao_tht:DIP-14_W7.62mm_Socket_LongPads, B.Cu at (91.1, 110.2)
- added U3: TL072, ao_tht:DIP-8_W7.62mm_Socket_LongPads, B.Cu at (116.5, 114.0)
Routing:
- net -12V: track 0.00 -> 206.6 mm, vias 0 -> 1
- net +12V: track 0.00 -> 168.3 mm, vias 0 -> 1
- net Net-(C14-Pad2): track 0.00 -> 138.2 mm
- net Net-(C12-Pad2): track 0.00 -> 132.9 mm
- net /Summers/+10V: track 0.00 -> 128.8 mm
- net /Summers/IN_2_1_WIP: track 0.00 -> 124.6 mm
- net /Summers/IN2_1: track 0.00 -> 109.9 mm
- net /Summers/IN2_2: track 0.00 -> 104.6 mm
- net /Summers/IN1_3: track 0.00 -> 68.3 mm
- net /Summers/IN1_4: track 0.00 -> 59.5 mm
- net /Linear and RC lag/IN_LAG_B: track 0.00 -> 57.9 mm, vias 0 -> 1
- net /Linear and RC lag/LAG_RC_WIP: track 0.00 -> 55.1 mm
- net /Linear and RC lag/LIN_IN: track 0.00 -> 54.8 mm
- net Net-(C11-Pad2): track 0.00 -> 50.8 mm
- net /Linear and RC lag/LIN_SPEED: track 0.00 -> 50.1 mm
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- added copper zone on B.Cu, net GND
- added copper zone on F.Cu, net GND
- added copper zone on B.Cu, net GND1
- added copper zone on F.Cu, net GND1
Other:
- board outline added: 171 x 174 mm
- net class Default removed
- net class Power removed
