File: Hardware/PCB/voltproc/voltproc.kicad_pcb (KiCad board)
At the start: 2 copper layers, 171 x 174 mm, 77 parts, among them J1 Synth_power_2x5, J10 Jack, J11 Jack, J12 Jack, J13 Jack, J14 Jack, J15 Jack, J16 Jack, J17 Jack, J18 Jack, J19 Jack, J2 2_pin_Molex_header, J3 2_pin_Molex_header, J4 Conn_01x13, J7 Conn_01x13, J8 Jack, J9 Jack, SW1 SW_DPDT_x2, SW2 SW_DPDT_x2, U1 TL074, U2 TL074, U3 TL072

Commit message: Redo layout
Parts:
- C11, C12, C3: footprint ao_tht:C_Disc_D3.0mm_W1.6mm_P2.50mm -> ao_tht:C_Disc_D5.0mm_W2.5mm_P5.00mm
- C4: footprint ao_tht:C_Disc_D3.0mm_W1.6mm_P2.50mm -> ao_tht:C_Rect_L7.2mm_W2.5mm_P5.00mm_FKS2_FKP2_MKS2_MKP2
- C6: footprint ao_tht:C_Disc_D3.0mm_W1.6mm_P2.50mm -> ao_tht:C_Rect_L7.2mm_W4.5mm_P5.00mm_FKS2_FKP2_MKS2_MKP2
- moved R20 64.3 mm to (130.5, 23.8), turned to 180 degrees
- moved R25 61.8 mm to (130.5, 39.0), turned to 180 degrees
- moved R21 61.2 mm to (130.5, 31.4), turned to 180 degrees
- moved J1 57.2 mm to (70.8, 34.6)
- moved C12 55.8 mm to (125.4, 20.0)
- moved C14 52.3 mm to (122.9, 46.7), turned to 180 degrees
- moved RV1 50.0 mm to (175.0, 119.0)
- moved RV4 50.0 mm to (225.0, 119.0)
- moved C16 45.7 mm to (122.8, 35.2), turned to 180 degrees
- moved R27 44.4 mm to (120.3, 42.9), turned to 0 degrees
- moved R23 42.6 mm to (120.3, 27.6), turned to 0 degrees
- moved D2 38.1 mm to (81.0, 24.2), turned to 0 degrees
- moved R28 32.5 mm to (105.1, 20.0), turned to 180 degrees
- moved J2 32.4 mm to (84.1, 45.4)
- moved R19 28.4 mm to (91.1, 36.5)
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Routing:
- net /Summers/IN2_1: track 109.9 -> 172.1 mm
- net /Summers/OUT1: track 8.02 -> 61.3 mm, vias 0 -> 1
- net -12V: track 206.6 -> 249.8 mm, vias 1 -> 2
- net +12V: track 168.3 -> 210.7 mm, vias 1 -> 2
- net Net-(C12-Pad2): track 132.9 -> 169.3 mm
- net /Summers/IN1_1: track 44.9 -> 11.6 mm
- net /Summers/IN2_2: track 104.6 -> 73.4 mm
- net /Summers/IN_2_1_WIP: track 124.6 -> 95.8 mm
- net /Summers/~{OUT1}: track 48.4 -> 75.7 mm, vias 0 -> 1
- net /Summers/IN1_3: track 68.3 -> 48.0 mm
- net /Linear and RC lag/LIN_SPEED: track 50.1 -> 68.3 mm
- net /Linear and RC lag/LIN_OUT: track 49.1 -> 32.2 mm
- net /Linear and RC lag/RC_SPEED: track 43.4 -> 30.7 mm
- net Net-(C13-Pad2): track 36.8 -> 24.3 mm
- net /Summers/IN_1_2_WIP: track 22.0 -> 9.94 mm
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Other:
- outline, holes or cut-outs redrawn

Commit message: Redo layout
Parts:
- R29, TP1, TP2, TP3: moved to F.Cu
- moved C15 92.7 mm to (103.8, 127.9)
- moved C9 92.7 mm to (103.8, 25.1)
- moved R20 92.7 mm to (131.8, 116.5)
- moved U1 91.4 mm to (108.9, 134.3)
- moved R27 89.6 mm to (131.8, 131.8), turned to 180 degrees
- moved C12 88.9 mm to (126.6, 108.9), turned to 180 degrees
- moved C16 85.1 mm to (124.1, 120.3)
- moved U3 85.1 mm to (116.5, 28.9)
- moved R25 85.1 mm to (131.8, 124.1)
- moved C14 81.3 mm to (124.1, 127.9)
- moved R21 81.3 mm to (131.8, 112.7)
- moved C10 81.3 mm to (124.1, 40.3)
- moved R23 78.3 mm to (131.8, 105.1), turned to 180 degrees
- moved R29 50.6 mm to (120.3, 72.1), turned to 0 degrees
- moved R5 44.0 mm to (68.2, 106.3), turned to 0 degrees
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Connections:
- U1 pad 1: Net-(C11-Pad2) -> /Linear and RC lag/RC_OUT
- U1 pad 2: Net-(C11-Pad1) -> /Linear and RC lag/RC_OUT
- U1 pad 3: GND -> /Linear and RC lag/LAG_RC_WIP
- U1 pad 6: Net-(C13-Pad1) -> Net-(U1-Pad6)
- U1 pad 7: Net-(C13-Pad2) -> Net-(U1-Pad6)
- U3 pad 1: /Linear and RC lag/RC_OUT -> Net-(C11-Pad2)
- U3 pad 2: /Linear and RC lag/RC_OUT -> Net-(C11-Pad1)
- U3 pad 3: /Linear and RC lag/LAG_RC_WIP -> GND
- U3 pad 6: Net-(U3-Pad6) -> Net-(C13-Pad1)
- U3 pad 7: Net-(U3-Pad6) -> Net-(C13-Pad2)
Routing:
- net Net-(C14-Pad2): track 142.1 -> 21.6 mm
- net /Summers/IN2_1: track 172.1 -> 84.5 mm
- net Net-(C12-Pad2): track 169.3 -> 92.4 mm, vias 0 -> 1
- net /Summers/~{OUT1}: track 75.7 -> 19.3 mm, vias 1 -> 0
- net /Linear and RC lag/LIN_SPEED: track 68.3 -> 16.4 mm
- net /Linear and RC lag/LAG_OUT: track 50.4 -> 97.3 mm
- net /Linear and RC lag/LAG_LIN_CCW: track 51.3 -> 10.7 mm
- net Net-(C11-Pad2): track 44.6 -> 85.2 mm
- net /Summers/IN1_1: track 11.6 -> 50.0 mm
- net /Summers/IN1_3: track 48.0 -> 84.9 mm
- net /Summers/IN_2_1_WIP: track 95.8 -> 60.0 mm
- net /Linear and RC lag/IN_LAG_B: track 49.4 -> 83.3 mm
- net /Linear and RC lag/OUT_LAG_B: track 40.9 -> 7.79 mm
- net /Summers/OUT1: track 61.3 -> 28.3 mm, vias 1 -> 0
- net /Linear and RC lag/LIN_IN: track 51.1 -> 21.0 mm
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
Commit message: post breadboard revisions
Parts:
- added R32: 100k, ao_tht:R_Axial_DIN0207_L6.3mm_D2.5mm_P10.16mm_Horizontal, B.Cu at (93.7, 21.3)
- added R33: 100k, ao_tht:R_Axial_DIN0207_L6.3mm_D2.5mm_P10.16mm_Horizontal, B.Cu at (116.5, 72.1)
- added R34: 100k, ao_tht:R_Axial_DIN0207_L6.3mm_D2.5mm_P10.16mm_Horizontal, B.Cu at (121.6, 138.1)
- added R35: 100k, ao_tht:R_Axial_DIN0207_L6.3mm_D2.5mm_P10.16mm_Horizontal, B.Cu at (121.6, 100.0)
- C11, C12: footprint ao_tht:C_Disc_D5.0mm_W2.5mm_P5.00mm -> ao_tht:C_Disc_D3.0mm_W1.6mm_P2.50mm
- C13, C14: value 200pF -> 220pF
- C5: footprint ao_tht:C_Radial_D8.0mm_H11.5mm_P3.50mm -> ao_tht:C_Radial_D5.0mm_H11.0mm_P2.00mm
- C6: footprint ao_tht:C_Rect_L7.2mm_W4.5mm_P5.00mm_FKS2_FKP2_MKS2_MKP2 -> ao_tht:C_Rect_L7.2mm_W7.2mm_P5.00mm_FKS2_FKP2_MKS2_MKP2
- TP3: footprint ao_tht:TestPoint_THTPad_1.5x1.5mm_Drill0.7mm -> ao_tht:TestPoint_THTPad_D1.5mm_Drill0.7mm
- moved J2 12.7 mm to (108.9, 46.7)
- moved J3 12.7 mm to (116.5, 46.7)
- moved J7 5.06 mm to (203.9, 98.5)
- moved J4 5.06 mm to (103.9, 98.5)
- moved C4 4.51 mm to (101.2, 130.5)
- moved C15 1.82 mm to (105.1, 126.7), turned to 90 degrees
- moved R20 1.27 mm to (131.8, 115.2)
- moved R27 1.27 mm to (131.8, 130.5)
- moved R30 1.27 mm to (131.8, 134.3)
- moved TP1 1.27 mm to (102.5, 16.2)
- moved C12 1.27 mm to (126.6, 107.6)
- moved C14 1.27 mm to (124.1, 126.7)
- moved C16 1.27 mm to (124.1, 119.0)
- moved C6 1.27 mm to (101.2, 124.1)
- moved R21 1.27 mm to (131.8, 111.4)
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Connections:
- net /Summers/IN1_1 renamed /Summers/IN_1_1
- net /Summers/IN1_2 renamed /Summers/IN_1_2
- net /Summers/IN2_1 renamed /Summers/IN_2_2
- net /Summers/IN2_2 renamed /Summers/IN_2_1
- J4 pad 2: /Linear and RC lag/LIN_SPEED -> /Linear and RC lag/LAG_RC_WIP
- J4 pad 3: /Linear and RC lag/RC_SPEED -> /Linear and RC lag/LAG_LIN_CCW
- J4 pad 4: /Linear and RC lag/LAG_RC_WIP -> /Linear and RC lag/LAG_LIN_WIP
- J4 pad 5: /Linear and RC lag/LAG_LIN_CCW -> /Linear and RC lag/LIN_SPEED
- J4 pad 6: /Linear and RC lag/LAG_LIN_WIP -> /Linear and RC lag/RC_SPEED
- J7 pad 2: /Panel components/LIN_SPEED -> /Panel components/LAG_RC_WIP
- J7 pad 3: /Panel components/RC_SPEED -> /Panel components/LAG_LIN_CCW
- J7 pad 4: /Panel components/LAG_RC_WIP -> /Panel components/LAG_LIN_WIP
- J7 pad 5: /Panel components/LAG_LIN_CCW -> /Panel components/LIN_SPEED
- J7 pad 6: /Panel components/LAG_LIN_WIP -> /Panel components/RC_SPEED
Routing:
- net /Summers/IN_1_2: track 37.1 -> 19.9 mm
- net /Linear and RC lag/LIN_SPEED: track 16.4 -> 31.0 mm
- net /Summers/IN_1_1: track 50.0 -> 37.3 mm
- net /Panel components/LIN_IN: track 27.6 -> 37.9 mm
- net /Panel components/RC_SPEED: track 30.5 -> 39.1 mm
- net Net-(C11-Pad2): track 85.2 -> 93.2 mm
- net Net-(C14-Pad2): track 21.6 -> 29.5 mm
- net Net-(C13-Pad2): track 31.9 -> 39.6 mm
- net /Linear and RC lag/LAG_RC_WIP: track 53.9 -> 46.3 mm
- net /Summers/IN_1_1_WIP: track 11.2 -> 18.4 mm, vias 0 -> 1
- net /Linear and RC lag/LAG_LIN_CCW: track 10.7 -> 17.2 mm
- net /Panel components/LIN_SPEED: track 39.1 -> 45.2 mm
- net /Panel components/IN_2_1_CW: track 13.9 -> 7.82 mm
- net /Linear and RC lag/LAG_LIN_WIP: track 34.4 -> 39.9 mm
- net /Panel components/LIN_OUT: track 19.9 -> 25.3 mm
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Other:
- outline, holes or cut-outs redrawn

Commit message: Tidy up PCB
Parts:
- added GRAF2: CC0 logo, ao_tht:CC0_logo, B.Cu at (85.0, 145.0)
- added GRAF3: AO logo, ao_tht:analogoutput, B.Cu at (84.2, 47.5)
- R29: moved to B.Cu
- moved J12 25.0 mm to (75.1, 150.0)
- moved J15 25.0 mm to (75.0, 175.0)
- moved C14 7.62 mm to (131.8, 126.7)
- moved C16 7.62 mm to (124.1, 126.7)
- moved R27 3.81 mm to (131.8, 134.3)
- moved R30 3.81 mm to (131.8, 130.5)
Connections:
- net /Summers/IN_1_1 renamed /Summers/IN_1_1_CW
- net /Summers/IN_1_2 renamed /Summers/IN_1_2_CW
- net /Summers/IN_2_1 renamed /Summers/IN_2_1_CW
Routing:
- net /Summers/IN_2_1_CW: track 74.3 -> 49.2 mm
- net /Summers/+10V: track 127.3 -> 102.4 mm
- net Net-(C14-Pad1): track 23.8 -> 36.6 mm
- net /Summers/IN_2_2: track 84.3 -> 95.8 mm
- net -12V: track 227.3 -> 222.6 mm
- net Net-(C14-Pad2): track 29.5 -> 25.5 mm
- net Net-(C12-Pad1): track 25.6 -> 28.7 mm
- net /Summers/OUT2: track 25.9 -> 27.5 mm
- net Net-(C12-Pad2): track 95.1 -> 96.7 mm, vias 1 -> 0
- net /Linear and RC lag/LAG_OUT: track 95.2 -> 96.0 mm
- net /Linear and RC lag/LIN_OUT: track 33.9 -> 34.5 mm
Other:
- board text added: "IN_1_1"
- board text added: "IN_1_1 POT WIP / CW"
- board text added: "IN_1_2"
- board text added: "IN_1_2 POT WIP / CW"
- board text added: "IN_1_3"
- board text added: "IN_1_4"
- board text added: "IN_2_1"
- board text added: "IN_2_1 POT"
- board text added: "IN_2_2"
- board text added: "IN_LAG"
- board text added: "LAG POT"
- board text added: "LAG RC/LIN"
- board text added: "LAG SPEED"
- board text added: "Main board"
- board text added: "OUT1"
- board text added: "OUT2"
- board text added: "OUT_LAG"
- board text added: "VOLTAGE PROCESSOR 7/2022 Rich Holmes CC0 https://github.com/holmesrichards/voltproc"
- board text added: "VOLTAGE PROCESSOR Controls board"
- board text added: "~{OUT1}"
- board text added: "~{OUT2}"

Commit message: CC0 add version
Other:
- board text added: "VOLTAGE PROCESSOR 7/2022 Rich Holmes CC0 1.0 https://github.com/holmesrichards/voltproc"
- board text removed: "VOLTAGE PROCESSOR 7/2022 Rich Holmes CC0 https://github.com/holmesrichards/voltproc"
Changed lines of the file:
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@@
     (effects (font (size 1 1) (thickness 0.15)) (justify mirror))
   )
-  (gr_text "VOLTAGE PROCESSOR\n7/2022 Rich Holmes CC0\nhttps://github.com/holmesrichards/voltproc" (at 83.998 137.592) (layer "B.SilkS")
+  (gr_text "VOLTAGE PROCESSOR\n7/2022 Rich Holmes CC0 1.0\nhttps://github.com/holmesrichards/voltproc" (at 83.998 137.592) (layer "B.SilkS")
     (effects (font (size 1 1) (thickness 0.15)) (justify mirror))
   )

Commit message: Pre fab tweaks, Gerbers, cap descriptions
Parts:
- added B1: Board, ao_tht:Board_Marker, F.Cu at (98.0, 14.0)
- added B2: Board, ao_tht:Board_Marker, F.Cu at (200.0, 95.5)
- J2, J3: value 2_pin_Molex_header -> 3_pin_Molex_header; footprint ao_tht:Molex_KK-254_AE-6410-02A_1x02_P2.54mm_Vertical -> ao_tht:Molex_KK-254_AE-6410-03A_1x03_P2.54mm_Vertical
- moved J2 5.08 mm to (103.8, 46.7)
- moved R32 3.81 mm to (93.7, 40.3)
- moved J3 2.54 mm to (114.0, 46.7)
- renumbered C16 to C10, C9 to C15, C10 to C16, C15 to C9, R32 to R28, R33 to R29, R34 to R30, R35 to R31, R28 to R32, R29 to R33, R30 to R34, R31 to R35, RV1 to RV3, U2 to U1, U1 to U2
Connections:
- J2 pad 1: /Summers/IN_1_1_CW -> GND
- J3 pad 1: /Summers/IN_1_2_CW -> GND
Routing:
- net /Summers/IN1_4: track 69.9 -> 73.8 mm
- net +12V: track 197.7 -> 193.8 mm
- net Net-(C13-Pad2): track 39.6 -> 35.8 mm
- net /Summers/IN_1_1_WIP: track 18.4 -> 21.1 mm
- net /Summers/IN_1_2_CW: track 19.9 -> 22.4 mm
- net /Summers/IN_1_2_WIP: track 23.8 -> 26.4 mm
- net /Summers/OUT1: track 27.7 -> 29.7 mm
- net Net-(C11-Pad2): track 93.2 -> 95.1 mm
- net -12V: track 222.6 -> 224.0 mm
- net /Linear and RC lag/LIN_OUT: track 34.5 -> 33.5 mm
Other:
- outline, holes or cut-outs redrawn
- board text added: "IN_1_1 POT CW/WIP/GND"
- board text added: "IN_1_2 POT CW/WIP/GND"
- board text added: "VOLTAGE PROCESSOR 7/2022 Rich Holmes CC0 1.0 from ARP and MFOS designs https://github.com/holmesrichards/voltproc"
- board text removed: "IN_1_1 POT WIP / CW"
- board text removed: "IN_1_2 POT WIP / CW"
- board text removed: "VOLTAGE PROCESSOR 7/2022 Rich Holmes CC0 1.0 https://github.com/holmesrichards/voltproc"
