File: Hardware/PCB/voltproc/voltproc.kicad_sch (KiCad schematic)
At the start: 15 parts, among them J1 Synth_power_2x5, J2 2_pin_Molex_header, J3 2_pin_Molex_header, J4 Conn_01x13, J5 2_pin_Molex_connector, J6 2_pin_Molex_connector, J7 Conn_01x13

Commit message: Redo layout
Parts:
- C1, C2: value 10uF -> (none); footprint ao_tht:CP_Radial_D6.3mm_P2.50mm -> (none)
- D1, D2: value 1N5817 -> (none); footprint ao_tht:D_DO-41_SOD81_P10.16mm_Horizontal -> (none)
- GRAF1: value Holes -> (none); footprint voltproc:voltproc_panel_holes -> (none)
- J1: value Synth_power_2x5 -> (none); footprint ao_tht:Power_Header -> (none)
- J2, J3: value 2_pin_Molex_header -> (none); footprint ao_tht:Molex_KK-254_AE-6410-02A_1x02_P2.54mm_Vertical -> (none)
- J4: value Conn_01x13 -> (none); footprint Connector_PinHeader_2.54mm:PinHeader_1x13_P2.54mm_Vertical -> (none)
- J5, J6: value 2_pin_Molex_connector -> (none); footprint ao_tht:Molex_KK-254_AE-6410-02A_1x02_P2.54mm_Vertical -> (none)
- J7: value Conn_01x13 -> (none); footprint Connector_PinSocket_2.54mm:PinSocket_1x13_P2.54mm_Vertical -> (none)
- TP1: value -12V -> (none); footprint ao_tht:TestPoint_THTPad_D1.5mm_Drill0.7mm -> (none)
- TP2: value +12V -> (none); footprint ao_tht:TestPoint_THTPad_D1.5mm_Drill0.7mm -> (none)
- TP3: value GND -> (none); footprint ao_tht:TestPoint_THTPad_1.5x1.5mm_Drill0.7mm -> (none)
Changed lines of the file:
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@@
     (in_bom yes) (on_board yes)
     (property "Reference" "D1" (id 0) (at 76.2 167.2336 0))
-    (property "Value" "1N5817" (id 1) (at 76.2 169.545 0))
-    (property "Footprint" "ao_tht:D_DO-41_SOD81_P10.16mm_Horizontal" (id 2) (at 76.2 172.72 0)
+    (property "Value" "" (id 1) (at 76.2 169.545 0))
+    (property "Footprint" "" (id 2) (at 76.2 172.72 0)
       (effects (font (size 1.27 1.27)) hide)
     )
@@
       (effects (font (size 1.27 1.27)) (justify left))
     )
-    (property "Value" "10uF" (id 1) (at 105.8672 173.863 0)
-      (effects (font (size 1.27 1.27)) (justify left))
-    )
-    (property "Footprint" "ao_tht:CP_Radial_D6.3mm_P2.50mm" (id 2) (at 103.8352 176.53 0)
+    (property "Value" "" (id 1) (at 105.8672 173.863 0)
+      (effects (font (size 1.27 1.27)) (justify left))
+    )
+    (property "Footprint" "" (id 2) (at 103.8352 176.53 0)
       (effects (font (size 1.27 1.27)) hide)
     )
@@
       (effects (font (size 1.524 1.524)))
     )
-    (property "Value" "Synth_power_2x5" (id 1) (at 46.99 169.1386 0)
+    (property "Value" "" (id 1) (at 46.99 169.1386 0)
       (effects (font (size 1.524 1.524)))
     )
-    (property "Footprint" "ao_tht:Power_Header" (id 2) (at 46.99 177.8 0)
+    (property "Footprint" "" (id 2) (at 46.99 177.8 0)
       (effects (font (size 1.524 1.524)) hide)
     )
@@
     (in_bom yes) (on_board yes)
     (property "Reference" "D2" (id 0) (at 76.2 177.3936 0))
-    (property "Value" "1N5817" (id 1) (at 76.2 179.705 0))
-    (property "Footprint" "ao_tht:D_DO-41_SOD81_P10.16mm_Horizontal" (id 2) (at 76.2 182.88 0)
+    (property "Value" "" (id 1) (at 76.2 179.705 0))
+    (property "Footprint" "" (id 2) (at 76.2 182.88 0)
       (effects (font (size 1.27 1.27)) hide)
     )
@@
       (effects (font (size 1.27 1.27)) (justify left))
     )
-    (property "Value" "10uF" (id 1) (at 105.8672 181.483 0)
-      (effects (font (size 1.27 1.27)) (justify left))
-    )
-    (property "Footprint" "ao_tht:CP_Radial_D6.3mm_P2.50mm" (id 2) (at 103.8352 184.15 0)
+    (property "Value" "" (id 1) (at 105.8672 181.483 0)
+      (effects (font (size 1.27 1.27)) (justify left))
+    )
+    (property "Footprint" "" (id 2) (at 103.8352 184.15 0)
       (effects (font (size 1.27 1.27)) hide)
     )
@@
       (effects (font (size 1.27 1.27)) (justify left))
     )
-    (property "Value" "2_pin_Molex_header" (id 1) (at 87.63 64.77 0)
-      (effects (font (size 1.27 1.27)) (justify left))
-    )
-    (property "Footprint" "ao_tht:Molex_KK-254_AE-6410-02A_1x02_P2.54mm_Vertical" (id 2) (at 100.33 67.31 0)
+    (property "Value" "" (id 1) (at 87.63 64.77 0)
+      (effects (font (size 1.27 1.27)) (justify left))
+    )
+    (property "Footprint" "" (id 2) (at 100.33 67.31 0)
       (effects (font (size 1.27 1.27)) hide)
     )
@@
       (effects (font (size 1.27 1.27)) (justify left))
     )
-    (property "Value" "-12V" (id 1) (at 72.517 196.6846 0)
-      (effects (font (size 1.27 1.27)) (justify left))
-    )
-    (property "Footprint" "ao_tht:TestPoint_THTPad_D1.5mm_Drill0.7mm" (id 2) (at 76.2 198.12 0)
+    (property "Value" "" (id 1) (at 72.517 196.6846 0)
+      (effects (font (size 1.27 1.27)) (justify left))
+    )
+    (property "Footprint" "" (id 2) (at 76.2 198.12 0)
       (effects (font (size 1.27 1.27)) hide)
     )
@@
     (in_bom yes) (on_board no)
     (property "Reference" "J6" (id 0) (at 109.22 72.39 0))
-    (property "Value" "2_pin_Molex_connector" (id 1) (at 123.19 72.39 0))
-    (property "Footprint" "ao_tht:Molex_KK-254_AE-6410-02A_1x02_P2.54mm_Vertical" (id 2) (at 115.57 74.93 0)
+    (property "Value" "" (id 1) (at 123.19 72.39 0))
+    (property "Footprint" "" (id 2) (at 115.57 74.93 0)
       (effects (font (size 1.27 1.27)) hide)
     )
@@
     (in_bom yes) (on_board yes)
     (property "Reference" "J7" (id 0) (at 115.57 104.14 0))
-    (property "Value" "Conn_01x13" (id 1) (at 115.57 106.68 0))
-    (property "Footprint" "Connector_PinSocket_2.54mm:PinSocket_1x13_P2.54mm_Vertical" (id 2) (at 115.57 124.46 0)
+    (property "Value" "" (id 1) (at 115.57 106.68 0))
+    (property "Footprint" "" (id 2) (at 115.57 124.46 0)
       (effects (font (size 1.27 1.27)) hide)
     )
@@
       (effects (font (size 1.27 1.27)) (justify left))
     )
-    (property "Value" "Holes" (id 1) (at 136.525 174.4222 0)
-      (effects (font (size 1.27 1.27)) (justify left))
-    )
-    (property "Footprint" "voltproc:voltproc_panel_holes" (id 2) (at 129.54 172.72 0)
+    (property "Value" "" (id 1) (at 136.525 174.4222 0)
+      (effects (font (size 1.27 1.27)) (justify left))
+    )
+    (property "Footprint" "" (id 2) (at 129.54 172.72 0)
       (effects (font (size 1.27 1.27)) hide)
     )
@@
       (effects (font (size 1.27 1.27)) (justify left))
     )
-    (property "Value" "Conn_01x13" (id 1) (at 100.33 106.68 0))
-    (property "Footprint" "Connector_PinHeader_2.54mm:PinHeader_1x13_P2.54mm_Vertical" (id 2) (at 100.33 124.46 0)
+    (property "Value" "" (id 1) (at 100.33 106.68 0))
+    (property "Footprint" "" (id 2) (at 100.33 124.46 0)
       (effects (font (size 1.27 1.27)) hide)
     )
@@
       (effects (font (size 1.27 1.27)) (justify left))
     )
-    (property "Value" "GND" (id 1) (at 114.427 196.6846 0)
-      (effects (font (size 1.27 1.27)) (justify left))
-    )
-    (property "Footprint" "ao_tht:TestPoint_THTPad_1.5x1.5mm_Drill0.7mm" (id 2) (at 118.11 198.12 0)
+    (property "Value" "" (id 1) (at 114.427 196.6846 0)
+      (effects (font (size 1.27 1.27)) (justify left))
+    )
+    (property "Footprint" "" (id 2) (at 118.11 198.12 0)
       (effects (font (size 1.27 1.27)) hide)
     )
@@
       (effects (font (size 1.27 1.27)) (justify left))
     )
-    (property "Value" "+12V" (id 1) (at 92.837 196.6846 0)
-      (effects (font (size 1.27 1.27)) (justify left))
-    )
-    (property "Footprint" "ao_tht:TestPoint_THTPad_D1.5mm_Drill0.7mm" (id 2) (at 96.52 198.12 0)
+    (property "Value" "" (id 1) (at 92.837 196.6846 0)
+      (effects (font (size 1.27 1.27)) (justify left))
+    )
+    (property "Footprint" "" (id 2) (at 96.52 198.12 0)
       (effects (font (size 1.27 1.27)) hide)
     )
@@
       (effects (font (size 1.27 1.27)) (justify left))
     )
-    (property "Value" "2_pin_Molex_header" (id 1) (at 87.63 72.39 0)
-      (effects (font (size 1.27 1.27)) (justify left))
-    )
-    (property "Footprint" "ao_tht:Molex_KK-254_AE-6410-02A_1x02_P2.54mm_Vertical" (id 2) (at 100.33 74.93 0)
+    (property "Value" "" (id 1) (at 87.63 72.39 0)
+      (effects (font (size 1.27 1.27)) (justify left))
+    )
+    (property "Footprint" "" (id 2) (at 100.33 74.93 0)
       (effects (font (size 1.27 1.27)) hide)
     )
@@
     (in_bom yes) (on_board no)
     (property "Reference" "J5" (id 0) (at 109.22 64.77 0))
-    (property "Value" "2_pin_Molex_connector" (id 1) (at 123.19 64.77 0))
-    (property "Footprint" "ao_tht:Molex_KK-254_AE-6410-02A_1x02_P2.54mm_Vertical" (id 2) (at 115.57 67.31 0)
+    (property "Value" "" (id 1) (at 123.19 64.77 0))
+    (property "Footprint" "" (id 2) (at 115.57 67.31 0)
       (effects (font (size 1.27 1.27)) hide)
     )
@@
     )
     (path "/cb875800-6d8c-4644-8531-67cc7ba15934/2b720fb1-e4d7-4330-8853-46bab5b648ef"
-      (reference "C3") (unit 1) (value "47pF") (footprint "ao_tht:C_Disc_D3.0mm_W1.6mm_P2.50mm")
+      (reference "C3") (unit 1) (value "47pF") (footprint "ao_tht:C_Disc_D5.0mm_W2.5mm_P5.00mm")
     )
     (path "/cb875800-6d8c-4644-8531-67cc7ba15934/8fa4316a-8afd-41b9-b765-872dd31ac04b"
-      (reference "C4") (unit 1) (value "220nF") (footprint "ao_tht:C_Disc_D3.0mm_W1.6mm_P2.50mm")
+      (reference "C4") (unit 1) (value "220nF") (footprint "ao_tht:C_Rect_L7.2mm_W2.5mm_P5.00mm_FKS2_FKP2_MKS2_MKP2")
     )
     (path "/cb875800-6d8c-4644-8531-67cc7ba15934/0828935f-d307-4d83-83ac-e21d01b5dc8c"
@@
     )
     (path "/cb875800-6d8c-4644-8531-67cc7ba15934/3a2382be-9cb6-4f83-b279-a848ab520644"
-      (reference "C6") (unit 1) (value "1uF") (footprint "ao_tht:C_Disc_D3.0mm_W1.6mm_P2.50mm")
+      (reference "C6") (unit 1) (value "1uF") (footprint "ao_tht:C_Rect_L7.2mm_W4.5mm_P5.00mm_FKS2_FKP2_MKS2_MKP2")
     )
     (path "/cb875800-6d8c-4644-8531-67cc7ba15934/972312dd-5c5c-4577-b685-57af15d8bedd"
@@
     )
     (path "/37e25b07-cf59-45fe-844f-5417bc730cd4/19d769b5-2ef3-4fdb-a711-298b068871f5"
-      (reference "C11") (unit 1) (value "20pF") (footprint "ao_tht:C_Disc_D3.0mm_W1.6mm_P2.50mm")
+      (reference "C11") (unit 1) (value "20pF") (footprint "ao_tht:C_Disc_D5.0mm_W2.5mm_P5.00mm")
     )
     (path "/37e25b07-cf59-45fe-844f-5417bc730cd4/6e0b4302-d46b-471c-b060-79e2c3c8a5dd"
-      (reference "C12") (unit 1) (value "20pF") (footprint "ao_tht:C_Disc_D3.0mm_W1.6mm_P2.50mm")
+      (reference "C12") (unit 1) (value "20pF") (footprint "ao_tht:C_Disc_D5.0mm_W2.5mm_P5.00mm")
     )
     (path "/37e25b07-cf59-45fe-844f-5417bc730cd4/86315a7f-e7a3-40cb-b198-d482a34b711d"

Commit message: Redo layout
Parts:
- C1, C2: value (none) -> 10uF; footprint (none) -> ao_tht:CP_Radial_D6.3mm_P2.50mm
- D1, D2: value (none) -> 1N5817; footprint (none) -> ao_tht:D_DO-41_SOD81_P10.16mm_Horizontal
- GRAF1: value (none) -> Holes; footprint (none) -> voltproc:voltproc_panel_holes
- J1: value (none) -> Synth_power_2x5; footprint (none) -> ao_tht:Power_Header
- J2, J3: value (none) -> 2_pin_Molex_header; footprint (none) -> ao_tht:Molex_KK-254_AE-6410-02A_1x02_P2.54mm_Vertical
- J4: value (none) -> Conn_01x13; footprint (none) -> Connector_PinHeader_2.54mm:PinHeader_1x13_P2.54mm_Vertical
- J5, J6: value (none) -> 2_pin_Molex_connector; footprint (none) -> ao_tht:Molex_KK-254_AE-6410-02A_1x02_P2.54mm_Vertical
- J7: value (none) -> Conn_01x13; footprint (none) -> Connector_PinSocket_2.54mm:PinSocket_1x13_P2.54mm_Vertical
- TP1: value (none) -> -12V; footprint (none) -> ao_tht:TestPoint_THTPad_D1.5mm_Drill0.7mm
- TP2: value (none) -> +12V; footprint (none) -> ao_tht:TestPoint_THTPad_D1.5mm_Drill0.7mm
- TP3: value (none) -> GND; footprint (none) -> ao_tht:TestPoint_THTPad_1.5x1.5mm_Drill0.7mm

Commit message: post breadboard revisions
Parts:
- TP1, TP2: Config (none) -> DNF; now left out of the parts list
- TP3: footprint ao_tht:TestPoint_THTPad_1.5x1.5mm_Drill0.7mm -> ao_tht:TestPoint_THTPad_D1.5mm_Drill0.7mm; Config (none) -> DNF; now left out of the parts list
Connections:
- net Linear and RC lag/LAG_LIN_CCW: now also J4.3 (Pin_3); no longer J4.5 (Pin_5)
- net Linear and RC lag/LAG_LIN_WIP: now also J4.4 (Pin_4); no longer J4.6 (Pin_6)
- net Linear and RC lag/LAG_RC_WIP: now also J4.2 (Pin_2); no longer J4.4 (Pin_4)
- net Linear and RC lag/LIN_SPEED: now also J4.5 (Pin_5); no longer J4.2 (Pin_2)
- net Linear and RC lag/RC_SPEED: now also J4.6 (Pin_6); no longer J4.3 (Pin_3)
- net Panel components/LAG_LIN_CCW: now also J7.3 (Pin_3); no longer J7.5 (Pin_5)
- net Panel components/LAG_LIN_WIP: now also J7.4 (Pin_4); no longer J7.6 (Pin_6)
- net Panel components/LAG_RC_WIP: now also J7.2 (Pin_2); no longer J7.4 (Pin_4)
- net Panel components/LIN_SPEED: now also J7.5 (Pin_5); no longer J7.2 (Pin_2)
- net Panel components/RC_SPEED: now also J7.6 (Pin_6); no longer J7.3 (Pin_3)
- net Panel components/PANEL_GROUND renamed GND1
- net Summers/IN_1_1_CW renamed Summers/IN_1_1
- net Summers/IN_1_2_CW renamed Summers/IN_1_2
- net Summers/IN_2_1_CW renamed Summers/IN_2_1
Other:
- sheet Panel components ports: added none; removed PANEL_GROUND
- sheet Summers ports: added IN_1_1, IN_1_2, IN_2_1; removed IN_1_1_CW, IN_1_2_CW, IN_2_1_CW
- moved on the sheet: J2, J3, J4, J5, J6, J7

Commit message: Tidy up PCB
Parts:
- added GRAF2: CC0 logo, ao_tht:CC0_logo, symbol ao_symbols:Graphic
- added GRAF3: AO logo, ao_tht:analogoutput, symbol ao_symbols:Graphic
Connections:
- net Summers/IN_1_1 renamed Summers/IN_1_1_CW
- net Summers/IN_1_2 renamed Summers/IN_1_2_CW
- net Summers/IN_2_1 renamed Summers/IN_2_1_CW
Other:
- sheet Summers ports: added IN_1_1_CW, IN_1_2_CW, IN_2_1_CW; removed IN_1_1, IN_1_2, IN_2_1
Changed lines of the file:
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@@
     (pin "1")
+  )
+  (symbol (lib_id "ao_symbols:Graphic") (at 129.54 187.96 0) (unit 1)
+    (in_bom no) (on_board yes) (fields_autoplaced)
+    (property "Reference" "GRAF3" (id 0) (at 136.525 187.1253 0)
+      (effects (font (size 1.27 1.27)) (justify left))
+    )
+    (property "Value" "AO logo" (id 1) (at 136.525 189.6622 0)
+      (effects (font (size 1.27 1.27)) (justify left))
+    )
+    (property "Footprint" "ao_tht:analogoutput" (id 2) (at 129.54 187.96 0)
+      (effects (font (size 1.27 1.27)) hide)
+    )
+    (property "Datasheet" "" (id 3) (at 129.54 187.96 0)
+      (effects (font (size 1.27 1.27)) hide)
+    )
+    (property "Config" "DNF" (id 4) (at 129.54 187.96 0)
+      (effects (font (size 1.27 1.27)) hide)
+    )
   )
   (symbol (lib_id "Connector_Generic:Conn_01x13") (at 116.84 101.6 180) (unit 1)
@@
     (pin "9")
   )
+  (symbol (lib_id "ao_symbols:Graphic") (at 129.54 180.34 0) (unit 1)
+    (in_bom no) (on_board yes) (fields_autoplaced)
+    (property "Reference" "GRAF2" (id 0) (at 136.525 179.5053 0)
+      (effects (font (size 1.27 1.27)) (justify left))
+    )
+    (property "Value" "CC0 logo" (id 1) (at 136.525 182.0422 0)
+      (effects (font (size 1.27 1.27)) (justify left))
+    )
+    (property "Footprint" "ao_tht:CC0_logo" (id 2) (at 129.54 180.34 0)
+      (effects (font (size 1.27 1.27)) hide)
+    )
+    (property "Datasheet" "" (id 3) (at 129.54 180.34 0)
+      (effects (font (size 1.27 1.27)) hide)
+    )
+    (property "Config" "DNF" (id 4) (at 129.54 180.34 0)
+      (effects (font (size 1.27 1.27)) hide)
+    )
+  )
   (symbol (lib_id "ao_symbols:TestPoint") (at 113.03 198.12 0) (unit 1)
     (in_bom no) (on_board yes) (fields_autoplaced)
@@
       (effects (font (size 1.27 1.27)) (justify right))
     )
-    (pin "IN_2_1" output (at 76.2 73.66 0)
-      (effects (font (size 1.27 1.27)) (justify right))
-    )
-    (pin "IN_1_1" output (at 76.2 55.88 0)
-      (effects (font (size 1.27 1.27)) (justify right))
-    )
-    (pin "IN_1_2" output (at 76.2 63.5 0)
+    (pin "IN_2_1_CW" output (at 76.2 73.66 0)
+      (effects (font (size 1.27 1.27)) (justify right))
+    )
+    (pin "IN_1_1_CW" output (at 76.2 55.88 0)
+      (effects (font (size 1.27 1.27)) (justify right))
+    )
+    (pin "IN_1_2_CW" output (at 76.2 63.5 0)
       (effects (font (size 1.27 1.27)) (justify right))
     )
@@
       (reference "GRAF1") (unit 1) (value "Holes") (footprint "voltproc:voltproc_panel_holes")
     )
+    (path "/bc3a9f43-614d-4bb4-86c3-bd2d08f04422"
+      (reference "GRAF2") (unit 1) (value "CC0 logo") (footprint "ao_tht:CC0_logo")
+    )
+    (path "/50c42b8b-08f3-4420-a005-8a56543689fa"
+      (reference "GRAF3") (unit 1) (value "AO logo") (footprint "ao_tht:analogoutput")
+    )
     (path "/00000000-0000-0000-0000-00006074df58"

Commit message: Pre fab tweaks, Gerbers, cap descriptions
Parts:
- added B1: Board, ao_tht:Board_Marker, symbol ao_symbols:Board
- J2, J3: value 2_pin_Molex_header -> 3_pin_Molex_header; footprint ao_tht:Molex_KK-254_AE-6410-02A_1x02_P2.54mm_Vertical -> ao_tht:Molex_KK-254_AE-6410-03A_1x03_P2.54mm_Vertical; symbol ao_symbols:2_pin_Molex_header -> ao_symbols:3_pin_Molex_header; SKU A-804 -> A-805
- J5, J6: value 2_pin_Molex_connector -> 3_pin_Molex_connector; footprint ao_tht:Molex_KK-254_AE-6410-02A_1x02_P2.54mm_Vertical -> ao_tht:Molex_KK-254_AE-6410-03A_1x03_P2.54mm_Vertical; symbol ao_symbols:2_pin_Molex_connector -> ao_symbols:3_pin_Molex_connector; SKU A-826 -> A-827
Connections:
- net GND: now also J2.1 (Pin_1), J3.1 (Pin_1)
- net GND1: now also J5.1 (Pin_1), J6.1 (Pin_1)
- net Panel components/IN_1_1_CW: now also J5.3 (Pin_3); no longer J5.1 (Pin_1)
- net Panel components/IN_1_2_CW: now also J6.3 (Pin_3); no longer J6.1 (Pin_1)
- net Summers/IN_1_1_CW: now also J2.3 (Pin_3); no longer J2.1 (Pin_1)
- net Summers/IN_1_2_CW: now also J3.3 (Pin_3); no longer J3.1 (Pin_1)
