File: Hardware/PCB/voltproc/voltproc_panel.kicad_sch (KiCad schematic)
At the start: 6 parts, among them SW1 SW_DPDT_x2, SW2 SW_DPDT_x2

Commit message: Redo layout
Parts:
- RV1: value B100k -> (none); footprint ao_tht:Potentiometer_Alpha_16mm_Single_Vertical -> (none)
- RV2, RV3: value B100k -> (none)
- RV4: value B1M -> (none); footprint ao_tht:Potentiometer_Alpha_16mm_Dual_Vertical -> (none)
- SW1, SW2: value SW_DPDT_x2 -> (none); footprint ao_tht:DPDT-toggle-switch-1M-seriesx -> (none)
Changed lines of the file:
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@@
       (effects (font (size 1.27 1.27)) (justify right))
     )
-    (property "Value" "B100k" (id 1) (at 49.022 83.5022 0)
+    (property "Value" "" (id 1) (at 49.022 83.5022 0)
       (effects (font (size 1.27 1.27)) (justify right))
     )
@@
     (in_bom yes) (on_board yes) (fields_autoplaced)
     (property "Reference" "SW1" (id 0) (at 129.54 53.0692 0))
-    (property "Value" "SW_DPDT_x2" (id 1) (at 129.54 55.6061 0))
-    (property "Footprint" "ao_tht:DPDT-toggle-switch-1M-seriesx" (id 2) (at 129.54 59.69 0)
+    (property "Value" "" (id 1) (at 129.54 55.6061 0))
+    (property "Footprint" "" (id 2) (at 129.54 59.69 0)
       (effects (font (size 1.27 1.27)) hide)
     )
@@
       (effects (font (size 1.27 1.27)) (justify right))
     )
-    (property "Value" "B1M" (id 1) (at 49.022 134.1378 0)
-      (effects (font (size 1.27 1.27)) (justify right))
-    )
-    (property "Footprint" "ao_tht:Potentiometer_Alpha_16mm_Dual_Vertical" (id 2) (at 50.8 132.08 0)
+    (property "Value" "" (id 1) (at 49.022 134.1378 0)
+      (effects (font (size 1.27 1.27)) (justify right))
+    )
+    (property "Footprint" "" (id 2) (at 50.8 132.08 0)
       (effects (font (size 1.27 1.27)) hide)
     )
@@
     (in_bom yes) (on_board yes) (fields_autoplaced)
     (property "Reference" "SW2" (id 0) (at 129.54 86.0892 0))
-    (property "Value" "SW_DPDT_x2" (id 1) (at 129.54 88.6261 0))
-    (property "Footprint" "ao_tht:DPDT-toggle-switch-1M-seriesx" (id 2) (at 129.54 92.71 0)
+    (property "Value" "" (id 1) (at 129.54 88.6261 0))
+    (property "Footprint" "" (id 2) (at 129.54 92.71 0)
       (effects (font (size 1.27 1.27)) hide)
     )
@@
       (effects (font (size 1.27 1.27)) (justify right))
     )
-    (property "Value" "B1M" (id 1) (at 49.022 159.5378 0)
-      (effects (font (size 1.27 1.27)) (justify right))
-    )
-    (property "Footprint" "ao_tht:Potentiometer_Alpha_16mm_Dual_Vertical" (id 2) (at 50.8 157.48 0)
+    (property "Value" "" (id 1) (at 49.022 159.5378 0)
+      (effects (font (size 1.27 1.27)) (justify right))
+    )
+    (property "Footprint" "" (id 2) (at 50.8 157.48 0)
       (effects (font (size 1.27 1.27)) hide)
     )
@@
       (effects (font (size 1.27 1.27)) (justify right))
     )
-    (property "Value" "B100k" (id 1) (at 49.022 58.1022 0)
+    (property "Value" "" (id 1) (at 49.022 58.1022 0)
       (effects (font (size 1.27 1.27)) (justify right))
     )
@@
       (effects (font (size 1.27 1.27)) (justify right))
     )
-    (property "Value" "B100k" (id 1) (at 49.022 108.9022 0)
-      (effects (font (size 1.27 1.27)) (justify right))
-    )
-    (property "Footprint" "ao_tht:Potentiometer_Alpha_16mm_Single_Vertical" (id 2) (at 50.8 106.68 0)
+    (property "Value" "" (id 1) (at 49.022 108.9022 0)
+      (effects (font (size 1.27 1.27)) (justify right))
+    )
+    (property "Footprint" "" (id 2) (at 50.8 106.68 0)
       (effects (font (size 1.27 1.27)) hide)
     )
@@
     (in_bom yes) (on_board yes) (fields_autoplaced)
     (property "Reference" "SW1" (id 0) (at 129.54 70.8492 0))
-    (property "Value" "SW_DPDT_x2" (id 1) (at 129.54 73.3861 0))
-    (property "Footprint" "ao_tht:DPDT-toggle-switch-1M-seriesx" (id 2) (at 129.54 77.47 0)
+    (property "Value" "" (id 1) (at 129.54 73.3861 0))
+    (property "Footprint" "" (id 2) (at 129.54 77.47 0)
       (effects (font (size 1.27 1.27)) hide)
     )
@@
     (in_bom yes) (on_board yes) (fields_autoplaced)
     (property "Reference" "SW2" (id 0) (at 129.54 100.0592 0))
-    (property "Value" "SW_DPDT_x2" (id 1) (at 129.54 102.5961 0))
-    (property "Footprint" "ao_tht:DPDT-toggle-switch-1M-seriesx" (id 2) (at 129.54 106.68 0)
-      (effects (font (size 1.27 1.27)) hide)
-    )
+    (property "Value" "" (id 1) (at 129.54 102.5961 0))
+    (property "Footprint" "" (id 2) (at 129.54 106.68 0)
+      (effects (font (size 1.27 1.27)) hide)
+    )

Commit message: Redo layout
Parts:
- RV1: value (none) -> B100k; footprint (none) -> ao_tht:Potentiometer_Alpha_16mm_Single_Vertical
- RV2, RV3: value (none) -> B100k
- RV4: value (none) -> B1M; footprint (none) -> ao_tht:Potentiometer_Alpha_16mm_Dual_Vertical
- SW1, SW2: value (none) -> SW_DPDT_x2; footprint (none) -> ao_tht:DPDT-toggle-switch-1M-seriesx
Changed lines of the file:
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@@
       (effects (font (size 1.27 1.27)) (justify right))
     )
-    (property "Value" "" (id 1) (at 49.022 83.5022 0)
+    (property "Value" "B100k" (id 1) (at 49.022 83.5022 0)
       (effects (font (size 1.27 1.27)) (justify right))
     )
@@
     (in_bom yes) (on_board yes) (fields_autoplaced)
     (property "Reference" "SW1" (id 0) (at 129.54 53.0692 0))
-    (property "Value" "" (id 1) (at 129.54 55.6061 0))
-    (property "Footprint" "" (id 2) (at 129.54 59.69 0)
+    (property "Value" "SW_DPDT_x2" (id 1) (at 129.54 55.6061 0))
+    (property "Footprint" "ao_tht:DPDT-toggle-switch-1M-seriesx" (id 2) (at 129.54 59.69 0)
       (effects (font (size 1.27 1.27)) hide)
     )
@@
       (effects (font (size 1.27 1.27)) (justify right))
     )
-    (property "Value" "" (id 1) (at 49.022 134.1378 0)
-      (effects (font (size 1.27 1.27)) (justify right))
-    )
-    (property "Footprint" "" (id 2) (at 50.8 132.08 0)
+    (property "Value" "B1M" (id 1) (at 49.022 134.1378 0)
+      (effects (font (size 1.27 1.27)) (justify right))
+    )
+    (property "Footprint" "ao_tht:Potentiometer_Alpha_16mm_Dual_Vertical" (id 2) (at 50.8 132.08 0)
       (effects (font (size 1.27 1.27)) hide)
     )
@@
     (in_bom yes) (on_board yes) (fields_autoplaced)
     (property "Reference" "SW2" (id 0) (at 129.54 86.0892 0))
-    (property "Value" "" (id 1) (at 129.54 88.6261 0))
-    (property "Footprint" "" (id 2) (at 129.54 92.71 0)
+    (property "Value" "SW_DPDT_x2" (id 1) (at 129.54 88.6261 0))
+    (property "Footprint" "ao_tht:DPDT-toggle-switch-1M-seriesx" (id 2) (at 129.54 92.71 0)
       (effects (font (size 1.27 1.27)) hide)
     )
@@
       (effects (font (size 1.27 1.27)) (justify right))
     )
-    (property "Value" "" (id 1) (at 49.022 159.5378 0)
-      (effects (font (size 1.27 1.27)) (justify right))
-    )
-    (property "Footprint" "" (id 2) (at 50.8 157.48 0)
+    (property "Value" "B1M" (id 1) (at 49.022 159.5378 0)
+      (effects (font (size 1.27 1.27)) (justify right))
+    )
+    (property "Footprint" "ao_tht:Potentiometer_Alpha_16mm_Dual_Vertical" (id 2) (at 50.8 157.48 0)
       (effects (font (size 1.27 1.27)) hide)
     )
@@
       (effects (font (size 1.27 1.27)) (justify right))
     )
-    (property "Value" "" (id 1) (at 49.022 58.1022 0)
+    (property "Value" "B100k" (id 1) (at 49.022 58.1022 0)
       (effects (font (size 1.27 1.27)) (justify right))
     )
@@
       (effects (font (size 1.27 1.27)) (justify right))
     )
-    (property "Value" "" (id 1) (at 49.022 108.9022 0)
-      (effects (font (size 1.27 1.27)) (justify right))
-    )
-    (property "Footprint" "" (id 2) (at 50.8 106.68 0)
+    (property "Value" "B100k" (id 1) (at 49.022 108.9022 0)
+      (effects (font (size 1.27 1.27)) (justify right))
+    )
+    (property "Footprint" "ao_tht:Potentiometer_Alpha_16mm_Single_Vertical" (id 2) (at 50.8 106.68 0)
       (effects (font (size 1.27 1.27)) hide)
     )
@@
     (in_bom yes) (on_board yes) (fields_autoplaced)
     (property "Reference" "SW1" (id 0) (at 129.54 70.8492 0))
-    (property "Value" "" (id 1) (at 129.54 73.3861 0))
-    (property "Footprint" "" (id 2) (at 129.54 77.47 0)
+    (property "Value" "SW_DPDT_x2" (id 1) (at 129.54 73.3861 0))
+    (property "Footprint" "ao_tht:DPDT-toggle-switch-1M-seriesx" (id 2) (at 129.54 77.47 0)
       (effects (font (size 1.27 1.27)) hide)
     )
@@
     (in_bom yes) (on_board yes) (fields_autoplaced)
     (property "Reference" "SW2" (id 0) (at 129.54 100.0592 0))
-    (property "Value" "" (id 1) (at 129.54 102.5961 0))
-    (property "Footprint" "" (id 2) (at 129.54 106.68 0)
-      (effects (font (size 1.27 1.27)) hide)
-    )
+    (property "Value" "SW_DPDT_x2" (id 1) (at 129.54 102.5961 0))
+    (property "Footprint" "ao_tht:DPDT-toggle-switch-1M-seriesx" (id 2) (at 129.54 106.68 0)
+      (effects (font (size 1.27 1.27)) hide)
+    )

Commit message: post breadboard revisions
Changed lines of the file:
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@@
     (comment 1 "or neighboring rights to this work. Published from United States.")
     (comment 2 "To the extent possible under law, Richard Holmes has waived all copyright and related ")
+    (comment 3 "Lag processor from MFOS design")
+    (comment 4 "From ARP 2600 schematics with updates and additions")
   )
   (junction (at 55.88 132.08) (diameter 0) (color 0 0 0 0)
-  )
-  (junction (at 50.8 177.8) (diameter 0) (color 0 0 0 0)
   )
   (junction (at 55.88 157.48) (diameter 0) (color 0 0 0 0)
@@
     (stroke (width 0) (type default) (color 0 0 0 0))
   )
-  (wire (pts (xy 54.61 177.8) (xy 50.8 177.8))
-    (stroke (width 0) (type default) (color 0 0 0 0))
-  )
   (wire (pts (xy 50.8 76.2) (xy 52.07 76.2))
     (stroke (width 0) (type default) (color 0 0 0 0))
@@
     (effects (font (size 1.27 1.27)) (justify left bottom))
   )
+  (label "RC_IN" (at 52.07 163.83 0)
+    (effects (font (size 1.27 1.27)) (justify left bottom))
+  )
   (label "RC_IN" (at 134.62 62.23 0)
     (effects (font (size 1.27 1.27)) (justify left bottom))
   )
-  (label "RC_IN" (at 52.07 163.83 0)
-    (effects (font (size 1.27 1.27)) (justify left bottom))
-  )
   (hierarchical_label "IN_2_1_CW" (shape output) (at 52.07 101.6 0)
     (effects (font (size 1.27 1.27)) (justify left))
@@
   )
   (hierarchical_label "IN_2_1_WIP" (shape output) (at 55.88 106.68 0)
-    (effects (font (size 1.27 1.27)) (justify left))
-  )
-  (hierarchical_label "PANEL_GROUND" (shape output) (at 54.61 177.8 0)
     (effects (font (size 1.27 1.27)) (justify left))
   )
@@
     (pin "6")
   )
-  (symbol (lib_name "R_POT_1") (lib_id "ao_symbols:R_POT") (at 50.8 55.88 0) (unit 1)
+  (symbol (lib_id "ao_symbols:R_POT") (at 50.8 55.88 0) (unit 1)
     (in_bom yes) (on_board no) (fields_autoplaced)
     (property "Reference" "RV2" (id 0) (at 49.022 55.3271 0)

Commit message: Pre fab tweaks, Gerbers, cap descriptions
Parts:
- added B2: Board, ao_tht:Board_Marker, symbol ao_symbols:Board
- renumbered RV2 to RV1, RV3 to RV2, RV1 to RV3
Changed lines of the file:
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@@
     (effects (font (size 1.27 1.27)) (justify left))
+  )
+  (symbol (lib_id "ao_symbols:Board") (at 128.905 135.255 0) (unit 1)
+    (in_bom no) (on_board yes) (fields_autoplaced)
+    (property "Reference" "B2" (id 0) (at 134.62 134.4203 0)
+      (effects (font (size 1.27 1.27)) (justify left))
+    )
+    (property "Value" "Board" (id 1) (at 134.62 136.9572 0)
+      (effects (font (size 1.27 1.27)) (justify left))
+    )
+    (property "Footprint" "ao_tht:Board_Marker" (id 2) (at 128.905 135.255 0)
+      (effects (font (size 1.27 1.27)) hide)
+    )
+    (property "Datasheet" "" (id 3) (at 128.905 135.255 0)
+      (effects (font (size 1.27 1.27)) hide)
+    )
+    (property "Config" "DNF" (id 4) (at 128.905 135.255 0)
+      (effects (font (size 1.27 1.27)) hide)
+    )
   )
   (symbol (lib_id "ao_symbols:R_POT") (at 50.8 81.28 0) (unit 1)
     (in_bom yes) (on_board no) (fields_autoplaced)
-    (property "Reference" "RV3" (id 0) (at 49.022 80.7271 0)
+    (property "Reference" "RV2" (id 0) (at 49.022 80.7271 0)
       (effects (font (size 1.27 1.27)) (justify right))
     )
@@
     )
     (property "Vendor" "Tayda" (id 4) (at 50.8 81.28 0)
+      (effects (font (size 1.27 1.27)) hide)
+    )
+    (property "Description" "Panel mount potentiometer" (id 5) (at 50.8 81.28 0)
       (effects (font (size 1.27 1.27)) hide)
     )
@@
   (symbol (lib_id "power:GND1") (at 50.8 177.8 0) (unit 1)
     (in_bom yes) (on_board yes) (fields_autoplaced)
-    (property "Reference" "#PWR043" (id 0) (at 50.8 184.15 0)
+    (property "Reference" "#PWR057" (id 0) (at 50.8 184.15 0)
       (effects (font (size 1.27 1.27)) hide)
     )
@@
       (effects (font (size 1.27 1.27)) hide)
     )
+    (property "Description" "Board mount vertical dual gang 16mm potentiometer" (id 4) (at 50.8 132.08 0)
+      (effects (font (size 1.27 1.27)) hide)
+    )
     (pin "1")
     (pin "2")
@@
   (symbol (lib_id "power:GND1") (at 50.8 60.96 0) (unit 1)
     (in_bom yes) (on_board yes) (fields_autoplaced)
-    (property "Reference" "#PWR040" (id 0) (at 50.8 67.31 0)
+    (property "Reference" "#PWR054" (id 0) (at 50.8 67.31 0)
       (effects (font (size 1.27 1.27)) hide)
     )
@@
   (symbol (lib_id "power:GND1") (at 50.8 86.36 0) (unit 1)
     (in_bom yes) (on_board yes) (fields_autoplaced)
-    (property "Reference" "#PWR041" (id 0) (at 50.8 92.71 0)
+    (property "Reference" "#PWR055" (id 0) (at 50.8 92.71 0)
       (effects (font (size 1.27 1.27)) hide)
     )
@@
   (symbol (lib_id "power:GND1") (at 138.43 91.44 0) (unit 1)
     (in_bom yes) (on_board yes) (fields_autoplaced)
-    (property "Reference" "#PWR044" (id 0) (at 138.43 97.79 0)
+    (property "Reference" "#PWR058" (id 0) (at 138.43 97.79 0)
       (effects (font (size 1.27 1.27)) hide)
     )
@@
       (effects (font (size 1.27 1.27)) hide)
     )
+    (property "Description" "Board mount vertical dual gang 16mm potentiometer" (id 4) (at 50.8 157.48 0)
+      (effects (font (size 1.27 1.27)) hide)
+    )
     (pin "1")
     (pin "2")
@@
   (symbol (lib_id "ao_symbols:R_POT") (at 50.8 55.88 0) (unit 1)
     (in_bom yes) (on_board no) (fields_autoplaced)
-    (property "Reference" "RV2" (id 0) (at 49.022 55.3271 0)
+    (property "Reference" "RV1" (id 0) (at 49.022 55.3271 0)
       (effects (font (size 1.27 1.27)) (justify right))
     )
@@
       (effects (font (size 1.27 1.27)) hide)
     )
+    (property "Description" "Panel mount potentiometer" (id 5) (at 50.8 55.88 0)
+      (effects (font (size 1.27 1.27)) hide)
+    )
     (pin "1")
     (pin "2")
@@
   (symbol (lib_id "power:GND1") (at 50.8 111.76 0) (unit 1)
     (in_bom yes) (on_board yes) (fields_autoplaced)
-    (property "Reference" "#PWR042" (id 0) (at 50.8 118.11 0)
+    (property "Reference" "#PWR056" (id 0) (at 50.8 118.11 0)
       (effects (font (size 1.27 1.27)) hide)
     )
@@
   (symbol (lib_id "ao_symbols:R_POT") (at 50.8 106.68 0) (unit 1)
     (in_bom yes) (on_board yes) (fields_autoplaced)
-    (property "Reference" "RV1" (id 0) (at 49.022 106.1271 0)
+    (property "Reference" "RV3" (id 0) (at 49.022 106.1271 0)
       (effects (font (size 1.27 1.27)) (justify right))
     )
@@
     )
     (property "Vendor" "Tayda" (id 4) (at 50.8 106.68 0)
+      (effects (font (size 1.27 1.27)) hide)
+    )
+    (property "Description" "Board mount vertical 16mm potentiometer" (id 5) (at 50.8 106.68 0)
       (effects (font (size 1.27 1.27)) hide)
     )
@@
   (symbol (lib_id "power:GND1") (at 138.43 105.41 0) (unit 1)
     (in_bom yes) (on_board yes) (fields_autoplaced)
-    (property "Reference" "#PWR045" (id 0) (at 138.43 111.76 0)
-      (effects (font (size 1.27 1.27)) hide)
-    )
+    (property "Reference" "#PWR059" (id 0) (at 138.43 111.76 0)
+      (effects (font (size 1.27 1.27)) hide)
+    )
