File: Hardware/PCB/voltproc/voltproc_summers.kicad_sch (KiCad schematic)
At the start: 37 parts, among them J10 Jack, J11 Jack, J12 Jack, J13 Jack, J14 Jack, J15 Jack, J16 Jack, J17 Jack, J18 Jack, J19 Jack, U1 TL074

Commit message: Redo layout
Parts:
- C11, C12: value 20pF -> (none); footprint ao_tht:C_Disc_D3.0mm_W1.6mm_P2.50mm -> (none)
- C13, C14: value 200pF -> (none); footprint ao_tht:C_Disc_D3.0mm_W1.6mm_P2.50mm -> (none)
- C15, C16: value 100nF -> (none); footprint ao_tht:C_Disc_D3.0mm_W1.6mm_P2.50mm -> (none)
- J10, J11, J12, J13, J14, J15, J16, J17, J18, J19: value Jack -> (none); footprint ao_tht:Jack_6.35mm_PJ_629HAN_slots -> (none)
- R12, R14: value 2.7k -> (none); footprint ao_tht:R_Axial_DIN0207_L6.3mm_D2.5mm_P10.16mm_Horizontal -> (none)
- R13, R15: value 15k -> (none); footprint ao_tht:R_Axial_DIN0207_L6.3mm_D2.5mm_P10.16mm_Horizontal -> (none)
- R16, R17, R18, R19, R20, R21, R22, R23: value 100k -> (none); footprint ao_tht:R_Axial_DIN0207_L6.3mm_D2.5mm_P10.16mm_Horizontal -> (none)
- R24, R25, R26, R27: value 10k -> (none); footprint ao_tht:R_Axial_DIN0207_L6.3mm_D2.5mm_P10.16mm_Horizontal -> (none)
- R28, R29, R30, R31: value 1k -> (none); footprint ao_tht:R_Axial_DIN0207_L6.3mm_D2.5mm_P10.16mm_Horizontal -> (none)
- U1: value TL074 -> (none); footprint ao_tht:DIP-14_W7.62mm_Socket_LongPads -> (none)

Commit message: Redo layout
Parts:
- removed C15, C16: (no value), symbol ao_symbols:C
- removed unit 1 of U1
- removed unit 2 of U1
- removed unit 5 of U1
- added C10, C9: 100nF, ao_tht:C_Disc_D3.0mm_W1.6mm_P2.50mm, symbol ao_symbols:C
- added U3: TL072, ao_tht:DIP-8_W7.62mm_Socket_LongPads, symbol ao_symbols:TL072
- C11, C12: value (none) -> 20pF; footprint (none) -> ao_tht:C_Disc_D5.0mm_W2.5mm_P5.00mm
- C13, C14: value (none) -> 200pF; footprint (none) -> ao_tht:C_Disc_D3.0mm_W1.6mm_P2.50mm
- J10, J11, J12, J13, J14, J15, J16, J17, J18, J19: value (none) -> Jack; footprint (none) -> ao_tht:Jack_6.35mm_PJ_629HAN_slots
- R12, R14: value (none) -> 2.7k; footprint (none) -> ao_tht:R_Axial_DIN0207_L6.3mm_D2.5mm_P10.16mm_Horizontal
- R13, R15: value (none) -> 15k; footprint (none) -> ao_tht:R_Axial_DIN0207_L6.3mm_D2.5mm_P10.16mm_Horizontal
- R16, R17, R18, R19, R20, R21, R22, R23: value (none) -> 100k; footprint (none) -> ao_tht:R_Axial_DIN0207_L6.3mm_D2.5mm_P10.16mm_Horizontal
- R24, R25, R26, R27: value (none) -> 10k; footprint (none) -> ao_tht:R_Axial_DIN0207_L6.3mm_D2.5mm_P10.16mm_Horizontal
- R28, R29, R30, R31: value (none) -> 1k; footprint (none) -> ao_tht:R_Axial_DIN0207_L6.3mm_D2.5mm_P10.16mm_Horizontal
- U1: value (none) -> TL074; footprint (none) -> ao_tht:DIP-14_W7.62mm_Socket_LongPads
Connections:
- net +12V: now also C9.1, U3.8 (V+)
- net -12V: now also C10.2, U3.4 (V-)
- net GND: now also C10.1, C9.2, U3.3 (+), U3.5 (+)
- net at C11.1, R16.2, R17.2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: now also U3.2 (-)
- net at C11.2, R22.2, R24.1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: now also U3.1
- net at C13.1, R24.2, R26.1: now also U3.6 (-)
- net at C13.2, R26.2, R28.1: now also U3.7

Commit message: post breadboard revisions
Parts:
- added R32, R33, R34, R35: 100k, ao_tht:R_Axial_DIN0207_L6.3mm_D2.5mm_P10.16mm_Horizontal, symbol ao_symbols:R
- C11, C12: footprint ao_tht:C_Disc_D5.0mm_W2.5mm_P5.00mm -> ao_tht:C_Disc_D3.0mm_W1.6mm_P2.50mm
- C13, C14: value 200pF -> 220pF
Connections:
- net GND: now also R32.2, R33.2, R34.2, R35.2
- net at C14.2, R27.2, R30.1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: now also R34.1
- net at C12.2, R23.2, R25.1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: now also R35.1
- net at C11.2, R22.2, R24.1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: now also R33.1
- net at C13.2, R26.2, R28.1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: now also R32.1
- net IN2_1 renamed IN_2_2
- net IN_1_1_CW renamed IN_1_1
- net IN_1_2_CW renamed IN_1_2
- net IN_2_1_CW renamed IN_2_1
Other:
- moved on the sheet: J16, J17, J18, J19, R28, R29, R30, R31

Commit message: Tidy up PCB
Connections:
- net IN_1_1 renamed IN_1_1_CW
- net IN_1_2 renamed IN_1_2_CW
- net IN_2_1 renamed IN_2_1_CW
Changed lines of the file:
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@@
     (effects (font (size 1.27 1.27)) (justify right))
   )
-  (hierarchical_label "IN_2_1" (shape output) (at 63.5 100.33 0)
+  (hierarchical_label "IN_2_1_CW" (shape output) (at 63.5 100.33 0)
     (effects (font (size 1.27 1.27)) (justify left))
   )
-  (hierarchical_label "IN_1_1" (shape output) (at 63.5 55.88 0)
+  (hierarchical_label "IN_1_1_CW" (shape output) (at 63.5 55.88 0)
     (effects (font (size 1.27 1.27)) (justify left))
   )
@@
     (effects (font (size 1.27 1.27)) (justify right))
   )
-  (hierarchical_label "IN_1_2" (shape output) (at 63.5 72.39 0)
+  (hierarchical_label "IN_1_2_CW" (shape output) (at 63.5 72.39 0)
     (effects (font (size 1.27 1.27)) (justify left))
   )

Commit message: Pre fab tweaks, Gerbers, cap descriptions
Parts:
- renumbered C9 to C15, C10 to C16, R32 to R28, R33 to R29, R34 to R30, R35 to R31, R28 to R32, R29 to R33, R30 to R34, R31 to R35, U1 to U2
