File: Hardware/Panel/voltproc_panel/voltproc_panel.kicad_pcb (KiCad board)
At the start: 2 copper layers, 75 x 200 mm, 23 parts

Commit message: Pre fab tweaks, Gerbers, cap descriptions
Other:
- board text added: "IN_1_1 CW/WIP/GND"
- board text added: "IN_1_2 CW/WIP/GND"
Changed lines of the file:
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@@
+    (effects (font (size 1 1) (thickness 0.15)) (justify mirror))
+  )
+  (gr_text "IN_1_1\nCW/WIP/GND" (at 28.6 46.1) (layer "B.SilkS")
+    (effects (font (size 1 1) (thickness 0.15)) (justify mirror))
+  )
+  (gr_text "IN_1_2\nCW/WIP/GND" (at 78.6 46.1) (layer "B.SilkS")
     (effects (font (size 1 1) (thickness 0.15)) (justify mirror))
   )
