File: Hardware/PCB/voltproc/Separate_PCBs/voltproc_b1.kicad_pcb (KiCad board)
At the start: 2 copper layers, 71 x 174 mm, 77 parts, among them J1 Synth_power_2x5, J10 Jack, J11 Jack, J12 Jack, J13 Jack, J14 Jack, J15 Jack, J16 Jack, J17 Jack, J18 Jack, J19 Jack, J2 3_pin_Molex_header, J3 3_pin_Molex_header, J4 Conn_01x13, J8 Jack, J9 Jack, U1 TL074, U2 TL074, U3 TL072

Commit message: gerbers
Parts:
- added B1: Board, ao_tht:Board_Marker, F.Cu at (48.5, 15.0)
Other:
- outline, holes or cut-outs redrawn

Commit message: final pre fab tweaks
Routing:
- net Board_0-/Summers/OUT1: track 29.7 -> 28.9 mm
Other:
- outline, holes or cut-outs redrawn

Commit message: R7->47k; documentation and photos
Parts:
- R7: value 4.7k -> 47k

Commit message: Glare at one nonconformist jack and make it behave
Parts:
- turned J17 to -90 degrees
Routing:
- net Board_0-/Summers/~{OUT1}: track 19.3 -> 9.02 mm
